File: other/KiCad_files/Overlord/Overlord.sch (KiCad schematic (older format))
At the start: 121 parts, among them J1 RJ45x2, J2 Screw_Terminal_01x09, J3 Screw_Terminal_01x09, J4 Screw_Terminal_01x09, J5 Screw_Terminal_01x09, J6 Screw_Terminal_01x09, J7 Conn_01x06_Male, Q1 2N7002E, Q2 2N7002E, Q3 2N7002E, Q4 2N7002E, Q5 2N7002E, Q6 2N7002E, U1 74HC4052D,653, U2 74HC4052D,653, U3 74HC4052D,653, U4 74HC4052D,653, U5 LM2575D2T-5G, U6 SN65HVD230, U7 MAX485ESA+T, U8 AP63203WU-7, U9 MAX485ESA+T

Commit message: Added LED pins for quick status display,  updated schematic (still need to update PCB),
Parts:
- removed C11: 1800uF, Capacitor_THT:C_Radial_D10.0mm_H20.0mm_P5.00mm, symbol Device:C
- removed D2, D3, D4, D5, D6: LED, LED_SMD:LED_0805_2012Metric, symbol Device:LED
- removed J3: Screw_Terminal_01x09, TerminalBlockCustom:TerminalBlock_9_5.08mm, symbol Connector:Screw_Terminal_01x09
- removed J7: Conn_01x06_Male, Connector_PinHeader_2.54mm:PinHeader_1x06_P2.54mm_Vertical, symbol Connector:Conn_01x06_Male
- removed Q5, Q6: 2N7002E, Package_TO_SOT_SMD:SOT-23, symbol Transistor_FET:2N7002E
- removed R19, R20: 1K, Resistor_SMD:R_1812_4532Metric_Pad1.30x3.40mm_HandSolder, symbol Device:R
- removed R21: V_select_12V, Resistor_SMD:R_1812_4532Metric_Pad1.30x3.40mm_HandSolder, symbol Device:R
- removed R22: V_select_5V, Resistor_SMD:R_1812_4532Metric_Pad1.30x3.40mm_HandSolder, symbol Device:R
- removed R23: V_select_3V3, Resistor_SMD:R_1812_4532Metric_Pad1.30x3.40mm_HandSolder, symbol Device:R
- removed R32, R34: 220, Resistor_SMD:R_1812_4532Metric_Pad1.30x3.40mm_HandSolder, symbol Device:R
- removed R35: 470R, Resistor_THT:R_Axial_DIN0207_L6.3mm_D2.5mm_P10.16mm_Horizontal, symbol Device:R
- added J3: Conn_01x12_Female, Connector_Molex:Molex_CLIK-Mate_502386-1270_1x12-1MP_P1.25mm_Horizontal, symbol Connector:Conn_01x12_Female
- added R5: 10K, Resistor_SMD:R_0805_2012Metric_Pad1.20x1.40mm_HandSolder, symbol Device:R
- R1, R2: value 35R -> 5K; footprint Resistor_THT:R_Axial_DIN0207_L6.3mm_D2.5mm_P10.16mm_Horizontal -> Resistor_SMD:R_0805_2012Metric_Pad1.20x1.40mm_HandSolder
- R15: value 1K -> 10K; footprint Resistor_SMD:R_1812_4532Metric_Pad1.30x3.40mm_HandSolder -> Resistor_SMD:R_0805_2012Metric_Pad1.20x1.40mm_HandSolder
- R16, R17, R18: value 1K -> 220; footprint Resistor_SMD:R_1812_4532Metric_Pad1.30x3.40mm_HandSolder -> Resistor_SMD:R_0805_2012Metric_Pad1.20x1.40mm_HandSolder
- R3: value 35R -> 10K; footprint Resistor_THT:R_Axial_DIN0207_L6.3mm_D2.5mm_P10.16mm_Horizontal -> Resistor_SMD:R_0805_2012Metric_Pad1.20x1.40mm_HandSolder
- R31, R33: value 220 -> 5K; footprint Resistor_SMD:R_1812_4532Metric_Pad1.30x3.40mm_HandSolder -> Resistor_SMD:R_0805_2012Metric_Pad1.20x1.40mm_HandSolder
- R4: value 120R -> 10K; footprint Resistor_THT:R_Axial_DIN0207_L6.3mm_D2.5mm_P10.16mm_Horizontal -> Resistor_SMD:R_0805_2012Metric_Pad1.20x1.40mm_HandSolder
Connections:
- net labels added: MB_A_1+, MB_B_1-, MB_DIR_CTRL_U1, MB_RX_U1, MB_TX_U1, STATUS_LED_B, STATUS_LED_G, STATUS_LED_R, UART_RX_0, UART_TX_0
- net labels removed: DEBUG_0, DEBUG_1, LP-LSD1, LP-LSD2, LP-LSD3, LP-LSD4, LP-LSD5, LP-LSD6, LPLSD_return, MB_A_0+, MB_B_0-, MB_DIR_CTRL_U0, MB_RX_U0, MB_TX_U0
- wire segments 598 -> 559
- no-connect marks 11 -> 13
Other:
- note added: "Connection interface"
- note added: "MODBUS transciever UART1\n"
- note removed: "Debug interface"
- note removed: "Low-power low side driver outputs"
- note removed: "MODBUS transciever UART0\n"
- note removed: "TODO: \n- change resistors for Modbus RJ LEDs as they are not bright enough / add transistors for that to not influence Modbus line too much\n- check if UART1 can be rerouted so that\nUART0 can still be used for normal UART operation\n- change RJ pins so that Modbus is on twisted pairs\n- add capacitors to OUTPUT transistors for better performance"
- moved on the sheet: 120R_enable1, C1, C12, C17, C2, C3, C4, C5, C6, D1, ESP1, J1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
