File: other/KiCad_files/Overlord/Overlord.kicad_pcb (KiCad board)
At the start: 2 copper layers, 155.7 x 86.3 mm, 298 parts, among them IC1 74HC4052D,653, IC2 74HC4052D,653, IC3 74HC4052D,653, IC4 74HC4052D,653, J1 39502-1011, J10 USB_B_Micro, J2 39502-1011, J3 39502-1011, J4 Conn_01x12_Pin, J5 Conn_01x10_Pin, J6 Conn_01x11_Pin, J7 Conn_01x11_Pin, U1 AP63203WU, U2 AP63205WU

Commit message: minor fixes for overlord interface,
Other:
- board text added: "MB_RX_2 MB_DIR_2 MB_TX_2 MB2_H MB2_L"
- board text removed: "MX_RX_2 MB_DIR_2 MB_TX_2 MB2_H MB2_L"
