File: other/KiCad_files/OverlordInterface/OverlordInterface/OverlordInterface.kicad_pcb (KiCad board)
At the start: 2 copper layers, 155 x 42 mm, 44 parts, among them J1 Conn_01x12_Pin, J2 DE9_Receptacle_MountingHoles_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, J3 DE9_Receptacle_MountingHoles_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, J4 DE9_Receptacle_MountingHoles_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, J5 DE9_Receptacle_MountingHoles_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

Commit message: minor fixes for overlord interface,
Other:
- board text added: "--- Overlord Interface --- Designed by Nimfrodian Ver 1.0 Rev D"
- board text added: "x x H x L x x x GND"
- board text added: "x x L H GND x x x x"
- board text added: "x x Tx x Rx x x x GND"
- board text removed: "--- Overlord Interface --- Designed by Nimfrodian Ver 1.0 Rev C"
